File: pcb/arty_s7_50_multi_net.sch (KiCad schematic (older format))
At the start: 19 parts, among them J1 01x04, J2 02x04, J3 02x06, J4 01x02, J5 02x08, J6 02x08, J7 02x06, U2 DP83848, U3 DP83848, U4 DP83848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

Commit message: fix for latest LiteX and SD-Card
Connections:
- net PX1 renamed CS_N
- net PX2 renamed MOSI
- net PX3 renamed MISO
- net PX4 renamed SCK
- net PX5 renamed DAT1
Changed lines of the file:
@@
 	600  5750 1450 5750
 Text Label 2400 2150 0    50   ~ 0
-PX1
+CS_N
 Text Label 2400 2250 0    50   ~ 0
-PX2
+MOSI
 Text Label 2400 3100 0    50   ~ 0
-PX3
+MISO
 Text Label 2400 3200 0    50   ~ 0
-PX4
+SCK
 Text Label 1400 3800 0    50   ~ 0
-PX5
+DAT1
 Text Label 1400 5250 0    50   ~ 0
-PX1
+CS_N
 Text Label 1400 5350 0    50   ~ 0
-PX2
+MOSI
 Text Label 1400 5450 0    50   ~ 0
-PX3
+MISO
 Text Label 1400 5550 0    50   ~ 0
-PX4
+SCK
 Wire Wire Line
 	2050 5250 2250 5250
 Text Label 2050 5250 0    50   ~ 0
-PX5
+DAT1
 Entry Wire Line
 	2250 5250 2350 5150
@@
 	9850 3450 10050 3450
 Connection ~ 9850 3450
+Wire Wire Line
+	3800 1400 3800 3450
 Wire Bus Line
 	10950 1900 10950 2300
@@
 Wire Bus Line
 	10950 2750 10950 4450
-Wire Wire Line
-	3800 1400 3800 3450
 $EndSCHEMATC
